File: Lab4/Lab4_Exercise/Lab4_Exercise.kicad_sch (KiCad schematic)
At the start: 6 parts, among them SW1 SW_SPDT

Commit message: Edited Lab 4 KiCAD files
Parts:
- removed BT1: 9V, symbol Device:Battery_Cell
- added J?: (no value), symbol Connector:Conn_01x02_Male
Connections:
- net GND: now reaches C1.2, D1.1 (K)
- net GND: now also J?.2 (Pin_2)
- net +9V: now reaches R1.1
- net +9V: now also J?.1 (Pin_1)
Changed lines of the file:
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@@
   (junction (at 154.94 84.455) (diameter 0) (color 0 0 0 0)
+  )
+  (junction (at 102.87 73.66) (diameter 0) (color 0 0 0 0)
+  )
+  (junction (at 102.87 78.74) (diameter 0) (color 0 0 0 0)
   )
   (wire (pts (xy 166.37 65.405) (xy 166.37 67.945))
@@
     (stroke (width 0) (type default) (color 0 0 0 0))
   )
-  (wire (pts (xy 106.045 70.485) (xy 106.045 62.865))
+  (wire (pts (xy 106.045 62.865) (xy 106.045 73.66))
     (stroke (width 0) (type default) (color 0 0 0 0))
   )
   (wire (pts (xy 154.94 65.405) (xy 166.37 65.405))
+    (stroke (width 0) (type default) (color 0 0 0 0))
+  )
+  (wire (pts (xy 102.87 63.5) (xy 102.87 73.66))
+    (stroke (width 0) (type default) (color 0 0 0 0))
+  )
+  (wire (pts (xy 102.87 73.66) (xy 106.045 73.66))
+    (stroke (width 0) (type default) (color 0 0 0 0))
+  )
+  (wire (pts (xy 102.87 78.74) (xy 102.87 80.645))
     (stroke (width 0) (type default) (color 0 0 0 0))
   )
@@
     (stroke (width 0) (type default) (color 0 0 0 0))
   )
+  (wire (pts (xy 102.87 78.74) (xy 106.045 78.74))
+    (stroke (width 0) (type default) (color 0 0 0 0))
+  )
   (wire (pts (xy 106.045 78.74) (xy 106.045 84.455))
     (stroke (width 0) (type default) (color 0 0 0 0))
   )
   (wire (pts (xy 154.94 77.47) (xy 154.94 84.455))
+    (stroke (width 0) (type default) (color 0 0 0 0))
+  )
+  (wire (pts (xy 102.87 80.645) (xy 103.505 80.645))
     (stroke (width 0) (type default) (color 0 0 0 0))
   )
@@
   )
   (wire (pts (xy 106.045 84.455) (xy 154.94 84.455))
+    (stroke (width 0) (type default) (color 0 0 0 0))
+  )
+  (wire (pts (xy 102.87 76.2) (xy 102.87 78.74))
     (stroke (width 0) (type default) (color 0 0 0 0))
   )
@@
     (pin "2")
   )
-  (symbol (lib_id "Device:Battery_Cell") (at 106.045 75.565 0) (unit 1)
+  (symbol (lib_id "Connector:Conn_01x02_Male") (at 97.79 73.66 0) (unit 1)
     (in_bom yes) (on_board yes) (fields_autoplaced)
-    (property "Reference" "BT1" (id 0) (at 109.22 72.2629 0)
-      (effects (font (size 1.27 1.27)) (justify left))
-    )
-    (property "Value" "9V" (id 1) (at 109.22 74.8029 0)
-      (effects (font (size 1.27 1.27)) (justify left))
-    )
-    (property "Footprint" "" (id 2) (at 106.045 74.041 90)
+    (property "Reference" "J?" (id 0) (at 98.425 68.58 0))
+    (property "Value" "" (id 1) (at 98.425 71.12 0))
+    (property "Footprint" "" (id 2) (at 97.79 73.66 0)
       (effects (font (size 1.27 1.27)) hide)
     )
-    (property "Datasheet" "~" (id 3) (at 106.045 74.041 90)
+    (property "Datasheet" "~" (id 3) (at 97.79 73.66 0)
       (effects (font (size 1.27 1.27)) hide)
     )
     (pin "1")
     (pin "2")
+  )
+  (symbol (lib_id "power:GND") (at 103.505 80.645 0) (unit 1)
+    (in_bom yes) (on_board yes) (fields_autoplaced)
+    (property "Reference" "#PWR?" (id 0) (at 103.505 86.995 0)
+      (effects (font (size 1.27 1.27)) hide)
+    )
+    (property "Value" "" (id 1) (at 103.505 85.09 0))
+    (property "Footprint" "" (id 2) (at 103.505 80.645 0)
+      (effects (font (size 1.27 1.27)) hide)
+    )
+    (property "Datasheet" "" (id 3) (at 103.505 80.645 0)
+      (effects (font (size 1.27 1.27)) hide)
+    )
+    (pin "1")
   )
   (symbol (lib_id "Switch:SW_SPDT") (at 141.605 62.865 0) (unit 1)
@@
     (pin "3")
   )
+  (symbol (lib_id "power:+9V") (at 102.87 63.5 0) (unit 1)
+    (in_bom yes) (on_board yes) (fields_autoplaced)
+    (property "Reference" "#PWR?" (id 0) (at 102.87 67.31 0)
+      (effects (font (size 1.27 1.27)) hide)
+    )
+    (property "Value" "" (id 1) (at 102.87 58.42 0))
+    (property "Footprint" "" (id 2) (at 102.87 63.5 0)
+      (effects (font (size 1.27 1.27)) hide)
+    )
+    (property "Datasheet" "" (id 3) (at 102.87 63.5 0)
+      (effects (font (size 1.27 1.27)) hide)
+    )
+    (pin "1")
+  )
   (sheet_instances
     (path "/" (page "1"))
   )
   (symbol_instances
-    (path "/cc8e3499-7dd5-4066-a137-f3cb9fc1ae50"
-      (reference "BT1") (unit 1) (value "9V") (footprint "")
+    (path "/db00ed9d-5cbd-42e1-a367-f32e41a8348a"
+      (reference "#PWR?") (unit 1) (value "GND") (footprint "")
+    )
+    (path "/ff3c247f-58c6-479d-ba30-61d36386d3d2"
+      (reference "#PWR?") (unit 1) (value "+9V") (footprint "")
     )
     (path "/8353e4b8-275c-410b-9cd5-0364950e6b19"
@@
       (reference "D1") (unit 1) (value "LED") (footprint "")
     )
+    (path "/a97d9593-88f3-490c-93d3-a1f528046ef8"
+      (reference "J?") (unit 1) (value "Conn_01x02_Male") (footprint "")
+    )
     (path "/a19b8e83-b1cc-49b8-b2c0-c5f45449f195"

Commit message: Added annotations
Parts:
- J1: renamed from J?; value (none) -> Conn_01x02_Male
Changed lines of the file:
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@@
   (symbol (lib_id "Connector:Conn_01x02_Male") (at 97.79 73.66 0) (unit 1)
     (in_bom yes) (on_board yes) (fields_autoplaced)
-    (property "Reference" "J?" (id 0) (at 98.425 68.58 0))
-    (property "Value" "" (id 1) (at 98.425 71.12 0))
+    (property "Reference" "J1" (id 0) (at 98.425 68.58 0))
+    (property "Value" "Conn_01x02_Male" (id 1) (at 98.425 71.12 0))
     (property "Footprint" "" (id 2) (at 97.79 73.66 0)
       (effects (font (size 1.27 1.27)) hide)
@@
   (symbol (lib_id "power:GND") (at 103.505 80.645 0) (unit 1)
     (in_bom yes) (on_board yes) (fields_autoplaced)
-    (property "Reference" "#PWR?" (id 0) (at 103.505 86.995 0)
+    (property "Reference" "#PWR02" (id 0) (at 103.505 86.995 0)
       (effects (font (size 1.27 1.27)) hide)
     )
-    (property "Value" "" (id 1) (at 103.505 85.09 0))
+    (property "Value" "GND" (id 1) (at 103.505 85.09 0))
     (property "Footprint" "" (id 2) (at 103.505 80.645 0)
       (effects (font (size 1.27 1.27)) hide)
@@
   (symbol (lib_id "power:+9V") (at 102.87 63.5 0) (unit 1)
     (in_bom yes) (on_board yes) (fields_autoplaced)
-    (property "Reference" "#PWR?" (id 0) (at 102.87 67.31 0)
+    (property "Reference" "#PWR01" (id 0) (at 102.87 67.31 0)
       (effects (font (size 1.27 1.27)) hide)
     )
-    (property "Value" "" (id 1) (at 102.87 58.42 0))
+    (property "Value" "+9V" (id 1) (at 102.87 58.42 0))
     (property "Footprint" "" (id 2) (at 102.87 63.5 0)
       (effects (font (size 1.27 1.27)) hide)
@@
   )
   (symbol_instances
+    (path "/ff3c247f-58c6-479d-ba30-61d36386d3d2"
+      (reference "#PWR01") (unit 1) (value "+9V") (footprint "")
+    )
     (path "/db00ed9d-5cbd-42e1-a367-f32e41a8348a"
-      (reference "#PWR?") (unit 1) (value "GND") (footprint "")
-    )
-    (path "/ff3c247f-58c6-479d-ba30-61d36386d3d2"
-      (reference "#PWR?") (unit 1) (value "+9V") (footprint "")
+      (reference "#PWR02") (unit 1) (value "GND") (footprint "")
     )
     (path "/8353e4b8-275c-410b-9cd5-0364950e6b19"
@@
     )
     (path "/a97d9593-88f3-490c-93d3-a1f528046ef8"
-      (reference "J?") (unit 1) (value "Conn_01x02_Male") (footprint "")
+      (reference "J1") (unit 1) (value "Conn_01x02_Male") (footprint "")
     )
     (path "/a19b8e83-b1cc-49b8-b2c0-c5f45449f195"
